Commit message: Updated camera params to switch to third-person

File: maze_gen/urdf/turtlebot3_burger.gazebo.xacro (robot description, xacro)
@@ -131,6 +131,6 @@
         <horizontal_fov>1.3962634</horizontal_fov>
         <image>
-          <width>800</width>
-          <height>800</height>
+          <width>1920</width>
+          <height>1080</height>
           <format>R8G8B8</format>
         </image>

File: maze_gen/urdf/turtlebot3_burger.urdf.xacro (robot description, xacro)
@@ -143,5 +143,5 @@
   <joint name="camera_joint" type="fixed">
     <axis xyz="0 1 0" />
-    <origin xyz="${camera_link} 0 1" rpy="0 0 0"/>
+    <origin xyz="${camera_link-0.5} 0 0.25" rpy="0 0 0"/>
     <parent link="base_link"/>
     <child link="camera_link"/>
@@ -149,5 +149,5 @@
   <!-- Camera -->
   <link name="camera_link">
-    <collision>
+    <!-- <collision>
       <origin xyz="0 0 0" rpy="0 0 0"/>
       <geometry>
@@ -166,5 +166,5 @@
       <origin xyz="0 0 0" rpy="0 0 0"/>
       <inertia ixx="1e-6" ixy="0" ixz="0" iyy="1e-6" iyz="0" izz="1e-6" />
-    </inertial>
+    </inertial> -->
   </link>
 </robot>
