Commit message: Move camera closer to robot
Doesn't start within wall

File: maze_gen/urdf/turtlebot3_burger.urdf.xacro (robot description, xacro)
@@ -143,5 +143,5 @@
   <joint name="camera_joint" type="fixed">
     <axis xyz="0 1 0" />
-    <origin xyz="${camera_link-0.5} 0 0.25" rpy="0 0 0"/>
+    <origin xyz="${camera_link-0.4} 0 0.25" rpy="0 0 0"/>
     <parent link="base_link"/>
     <child link="camera_link"/>
